File: PCB/V210/ChryslerScanner_V210/PowerSupply.kicad_sch (KiCad schematic)
At the start: 32 parts, among them J5 PROG EN, U5 SD8628, U6 TD1509, U7 TD1509P5, U8 AMS1117-3.3, U9 LM317_SOT-223

Commit message: WIP
Parts:
- C23, C25, C27, C28: footprint (none) -> Capacitor_SMD:C_0603_1608Metric
- D6: renamed from D14; value SS56 -> B560C-13-F; footprint (none) -> Diode_SMD:D_SMC; manf# (none) -> B560C-13-F
- D7: renamed from D15; value SS56 -> B560C-13-F; footprint (none) -> Diode_SMD:D_SMC; manf# (none) -> B560C-13-F
- D8: renamed from D16; value SS56 -> B560C-13-F; footprint (none) -> Diode_SMD:D_SMC; manf# (none) -> B560C-13-F
- D9: renamed from D17; value SS56 -> B560C-13-F; footprint (none) -> Diode_SMD:D_SMC; manf# (none) -> B560C-13-F
- J4: renamed from J5; footprint (none) -> Connector_PinHeader_2.54mm:PinHeader_1x02_P2.54mm_Vertical
- R27: renamed from R49; footprint (none) -> Resistor_SMD:R_0603_1608Metric
- R28: renamed from R50; footprint (none) -> Resistor_SMD:R_0603_1608Metric
- R29: renamed from R51; footprint (none) -> Resistor_SMD:R_0603_1608Metric
- R30: renamed from R52; footprint (none) -> Resistor_SMD:R_0603_1608Metric
- R31: renamed from R53; footprint (none) -> Resistor_SMD:R_0603_1608Metric
- R32: renamed from R54; footprint (none) -> Resistor_SMD:R_0603_1608Metric
- R33: renamed from R55; footprint (none) -> Resistor_SMD:R_0603_1608Metric
- R34: renamed from R56; footprint (none) -> Resistor_SMD:R_0603_1608Metric
- R35: renamed from R57; footprint (none) -> Resistor_SMD:R_0603_1608Metric
- U5: value SD8628 -> SDB628
- U8, U9: footprint Package_TO_SOT_SMD:SOT-223-3_TabPin2 -> (none)
Other:
- title: Chrysler Scanner -> TJ Diag
- moved on the sheet: C19, C20, C21, C22, C23, C24, C25, C26, C27, C28, D6, D7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
