File: PCB/V210/ChryslerScanner_V210/PowerSupply.kicad_sch (KiCad schematic)
At the start: 9 parts, among them U5 NCV7808BDTRKG, U6 TLV76150DCYR, U7 TLV76133DCYR

Commit message: WIP
Connections:
- net +12V: now also C20.1, U7.3 (VI)
- net GND: no longer C20.1, U7.3 (VI)
Changed lines of the file:
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@@
     (comment 3 "GPL V3 LICENSE")
   )
+  (junction (at 152.4 114.3) (diameter 0) (color 0 0 0 0)
+  )
   (junction (at 167.64 91.44) (diameter 0) (color 0 0 0 0)
   )
@@
   (junction (at 182.88 78.74) (diameter 0) (color 0 0 0 0)
   )
-  (junction (at 152.4 114.3) (diameter 0) (color 0 0 0 0)
-  )
   (junction (at 152.4 78.74) (diameter 0) (color 0 0 0 0)
   )
@@
     (stroke (width 0) (type default) (color 0 0 0 0))
   )
+  (wire (pts (xy 152.4 102.87) (xy 152.4 114.3))
+    (stroke (width 0) (type default) (color 0 0 0 0))
+  )
   (wire (pts (xy 182.88 114.3) (xy 182.88 118.11))
     (stroke (width 0) (type default) (color 0 0 0 0))
@@
   )
   (wire (pts (xy 152.4 91.44) (xy 167.64 91.44))
-    (stroke (width 0) (type default) (color 0 0 0 0))
-  )
-  (wire (pts (xy 152.4 91.44) (xy 152.4 114.3))
     (stroke (width 0) (type default) (color 0 0 0 0))
   )
@@
     (pin "2")
   )
+  (symbol (lib_id "power:+12V") (at 152.4 102.87 0) (unit 1)
+    (in_bom yes) (on_board yes) (fields_autoplaced)
+    (property "Reference" "#PWR?" (id 0) (at 152.4 106.68 0)
+      (effects (font (size 1.27 1.27)) hide)
+    )
+    (property "Value" "+12V" (id 1) (at 152.4 97.79 0))
+    (property "Footprint" "" (id 2) (at 152.4 102.87 0)
+      (effects (font (size 1.27 1.27)) hide)
+    )
+    (property "Datasheet" "" (id 3) (at 152.4 102.87 0)
+      (effects (font (size 1.27 1.27)) hide)
+    )
+    (pin "1")
+  )
   (symbol (lib_id "power:GND") (at 123.19 93.98 0) (unit 1)
