File: PCB/V210/ChryslerScanner_V210/VoltageSwitches.kicad_sch (KiCad schematic)
At the start: 44 parts

Commit message: Completed schematic.
Parts:
- gave numbers to parts that had none: 36

Commit message: WIP
Parts:
- removed Q10, Q11, Q12, Q13, Q6, Q7, Q8, Q9: HSW4602, Package_TO_SOT_SMD:SOT-23-6, symbol ChryslerScanner:HSW4602
- added Q10, Q11, Q12, Q13, Q6, Q7, Q8, Q9: DMC3025LSD-13, Package_SO:SO-8_3.9x4.9mm_P1.27mm, symbol ChryslerScanner:DMC3025LSD-13
- D10, D11, D12, D13, D6, D7, D8, D9: value MSK4005 -> STPS0540Z; footprint (none) -> Britishideas:SOD-123; manf# (none) -> STPS0540Z
- R30: renamed from R29; footprint (none) -> Resistor_SMD:R_0603_1608Metric
- R31: renamed from R30; footprint (none) -> Resistor_SMD:R_0603_1608Metric
- R32: renamed from R31; footprint (none) -> Resistor_SMD:R_0603_1608Metric
- R33: renamed from R32; footprint (none) -> Resistor_SMD:R_0603_1608Metric
- R34: renamed from R33; footprint (none) -> Resistor_SMD:R_0603_1608Metric
- R35: renamed from R34; footprint (none) -> Resistor_SMD:R_0603_1608Metric
- R36: renamed from R35; footprint (none) -> Resistor_SMD:R_0603_1608Metric
- R37: renamed from R36; footprint (none) -> Resistor_SMD:R_0603_1608Metric
- R38: renamed from R37; footprint (none) -> Resistor_SMD:R_0603_1608Metric
- R39: renamed from R38; footprint (none) -> Resistor_SMD:R_0603_1608Metric
- R40: renamed from R39; footprint (none) -> Resistor_SMD:R_0603_1608Metric
- R41: renamed from R40; footprint (none) -> Resistor_SMD:R_0603_1608Metric
- R42: renamed from R41; footprint (none) -> Resistor_SMD:R_0603_1608Metric
- R43: renamed from R42; footprint (none) -> Resistor_SMD:R_0603_1608Metric
- R44: renamed from R43; footprint (none) -> Resistor_SMD:R_0603_1608Metric
- R45: renamed from R44; footprint (none) -> Resistor_SMD:R_0603_1608Metric
- R46: renamed from R45; footprint (none) -> Resistor_SMD:R_0603_1608Metric
- R47: renamed from R46; footprint (none) -> Resistor_SMD:R_0603_1608Metric
- R48: renamed from R47; footprint (none) -> Resistor_SMD:R_0603_1608Metric
- R49: renamed from R48; footprint (none) -> Resistor_SMD:R_0603_1608Metric
Connections:
- net GND: now also Q10.1 (S), Q11.1 (S), Q12.1 (S), Q13.1 (S), Q6.1 (S), Q7.1 (S), Q8.1 (S), Q9.1 (S)
- net VAA: now also Q10.3 (1), Q12.3 (1), Q6.3 (1), Q8.3 (1)
- net VAA_TO_RX12: now also Q10.2 (G)
- net VAA_TO_RX14: now also Q12.2 (G)
- net VAA_TO_RX6: now also Q6.2 (G)
- net VAA_TO_RX9: now also Q8.2 (G)
- net VPP: now also Q11.3 (1), Q13.3 (1), Q7.3 (1), Q9.3 (1)
- net VPP_TO_RX12: now also Q11.2 (G)
- net VPP_TO_RX14: now also Q13.2 (G)
- net VPP_TO_RX6: now also Q7.2 (G)
- net VPP_TO_RX9: now also Q9.2 (G)
- net at R39.2: now also Q9.8 (D)
- net at R48.2, R49.1: now also Q13.4 (G)
- net at R37.2: now also Q8.4 (G), Q8.8 (D)
- net at R47.2: now also Q12.4 (G), Q12.8 (D)
- net at R42.2: now also Q10.4 (G), Q10.8 (D)
- net at D6.2 (A): now also Q6.5 (D)
- net at R33.2, R34.1: now also Q7.4 (G)
- net at D7.2 (A): now also Q7.5 (D)
- net at D11.2 (A): now also Q11.5 (D)
- net at D13.2 (A): now also Q13.5 (D)
- net at D8.2 (A): now also Q8.5 (D)
- net at R43.2, R44.1: now also Q11.4 (G)
- net at R44.2: now also Q11.8 (D)
- net at D10.2 (A): now also Q10.5 (D)
- net at R34.2: now also Q7.8 (D)
- net at D12.2 (A): now also Q12.5 (D)
- net at R32.2: now also Q6.4 (G), Q6.8 (D)
- net at R38.2, R39.1: now also Q9.4 (G)
- net at D9.2 (A): now also Q9.5 (D)
- net at R49.2: now also Q13.8 (D)
