File: PCB/V210/ChryslerScanner_V210/LEDs.kicad_sch (KiCad schematic)
At the start: 16 parts

Commit message: Completed schematic.
Parts:
- gave numbers to parts that had none: 16
Changed lines of the file:
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@@
   (symbol (lib_id "power:GND") (at 214.63 119.38 0) (unit 1)
     (in_bom yes) (on_board yes) (fields_autoplaced)
-    (property "Reference" "#PWR?" (id 0) (at 214.63 125.73 0)
+    (property "Reference" "#PWR034" (id 0) (at 214.63 125.73 0)
       (effects (font (size 1.27 1.27)) hide)
     )
@@
   (symbol (lib_id "power:GND") (at 171.45 119.38 0) (unit 1)
     (in_bom yes) (on_board yes) (fields_autoplaced)
-    (property "Reference" "#PWR?" (id 0) (at 171.45 125.73 0)
+    (property "Reference" "#PWR032" (id 0) (at 171.45 125.73 0)
       (effects (font (size 1.27 1.27)) hide)
     )
@@
   (symbol (lib_id "Device:R") (at 74.93 110.49 0) (unit 1)
     (in_bom yes) (on_board yes) (fields_autoplaced)
-    (property "Reference" "R?" (id 0) (at 77.47 109.2199 0)
+    (property "Reference" "R15" (id 0) (at 77.47 109.2199 0)
       (effects (font (size 1.27 1.27)) (justify left))
     )
@@
   (symbol (lib_id "Device:LED") (at 85.09 91.44 90) (unit 1)
     (in_bom yes) (on_board yes) (fields_autoplaced)
-    (property "Reference" "D?" (id 0) (at 88.9 91.7574 90)
+    (property "Reference" "D2" (id 0) (at 88.9 91.7574 90)
       (effects (font (size 1.27 1.27)) (justify right))
     )
@@
   (symbol (lib_id "Device:R") (at 161.29 110.49 0) (unit 1)
     (in_bom yes) (on_board yes) (fields_autoplaced)
-    (property "Reference" "R?" (id 0) (at 163.83 109.2199 0)
+    (property "Reference" "R19" (id 0) (at 163.83 109.2199 0)
       (effects (font (size 1.27 1.27)) (justify left))
     )
@@
   (symbol (lib_id "power:+5V") (at 214.63 74.93 0) (unit 1)
     (in_bom yes) (on_board yes) (fields_autoplaced)
-    (property "Reference" "#PWR?" (id 0) (at 214.63 78.74 0)
+    (property "Reference" "#PWR033" (id 0) (at 214.63 78.74 0)
       (effects (font (size 1.27 1.27)) hide)
     )
@@
   (symbol (lib_id "Transistor_FET:AO3400A") (at 82.55 102.87 0) (unit 1)
     (in_bom yes) (on_board yes) (fields_autoplaced)
-    (property "Reference" "Q?" (id 0) (at 88.9 101.5999 0)
+    (property "Reference" "Q2" (id 0) (at 88.9 101.5999 0)
       (effects (font (size 1.27 1.27)) (justify left))
     )
@@
   (symbol (lib_id "power:GND") (at 128.27 119.38 0) (unit 1)
     (in_bom yes) (on_board yes) (fields_autoplaced)
-    (property "Reference" "#PWR?" (id 0) (at 128.27 125.73 0)
+    (property "Reference" "#PWR030" (id 0) (at 128.27 125.73 0)
       (effects (font (size 1.27 1.27)) hide)
     )
@@
   (symbol (lib_id "Device:R") (at 85.09 81.28 0) (unit 1)
     (in_bom yes) (on_board yes) (fields_autoplaced)
-    (property "Reference" "R?" (id 0) (at 87.63 80.0099 0)
+    (property "Reference" "R16" (id 0) (at 87.63 80.0099 0)
       (effects (font (size 1.27 1.27)) (justify left))
     )
@@
   (symbol (lib_id "Transistor_FET:AO3400A") (at 168.91 102.87 0) (unit 1)
     (in_bom yes) (on_board yes) (fields_autoplaced)
-    (property "Reference" "Q?" (id 0) (at 175.26 101.5999 0)
+    (property "Reference" "Q4" (id 0) (at 175.26 101.5999 0)
       (effects (font (size 1.27 1.27)) (justify left))
     )
@@
   (symbol (lib_id "Transistor_FET:AO3400A") (at 212.09 102.87 0) (unit 1)
     (in_bom yes) (on_board yes) (fields_autoplaced)
-    (property "Reference" "Q?" (id 0) (at 218.44 101.5999 0)
+    (property "Reference" "Q5" (id 0) (at 218.44 101.5999 0)
       (effects (font (size 1.27 1.27)) (justify left))
     )
@@
   (symbol (lib_id "power:+5V") (at 85.09 74.93 0) (unit 1)
     (in_bom yes) (on_board yes) (fields_autoplaced)
-    (property "Reference" "#PWR?" (id 0) (at 85.09 78.74 0)
+    (property "Reference" "#PWR027" (id 0) (at 85.09 78.74 0)
       (effects (font (size 1.27 1.27)) hide)
     )
@@
   (symbol (lib_id "power:GND") (at 85.09 119.38 0) (unit 1)
     (in_bom yes) (on_board yes) (fields_autoplaced)
-    (property "Reference" "#PWR?" (id 0) (at 85.09 125.73 0)
+    (property "Reference" "#PWR028" (id 0) (at 85.09 125.73 0)
       (effects (font (size 1.27 1.27)) hide)
     )
@@
   (symbol (lib_id "Device:R") (at 214.63 81.28 0) (unit 1)
     (in_bom yes) (on_board yes) (fields_autoplaced)
-    (property "Reference" "R?" (id 0) (at 217.17 80.0099 0)
+    (property "Reference" "R22" (id 0) (at 217.17 80.0099 0)
       (effects (font (size 1.27 1.27)) (justify left))
     )
@@
   (symbol (lib_id "Device:R") (at 171.45 81.28 0) (unit 1)
     (in_bom yes) (on_board yes) (fields_autoplaced)
-    (property "Reference" "R?" (id 0) (at 173.99 80.0099 0)
+    (property "Reference" "R20" (id 0) (at 173.99 80.0099 0)
       (effects (font (size 1.27 1.27)) (justify left))
     )
@@
   (symbol (lib_id "Device:R") (at 118.11 110.49 0) (unit 1)
     (in_bom yes) (on_board yes) (fields_autoplaced)
-    (property "Reference" "R?" (id 0) (at 120.65 109.2199 0)
+    (property "Reference" "R17" (id 0) (at 120.65 109.2199 0)
       (effects (font (size 1.27 1.27)) (justify left))
     )
@@
   (symbol (lib_id "Device:LED") (at 128.27 91.44 90) (unit 1)
     (in_bom yes) (on_board yes) (fields_autoplaced)
-    (property "Reference" "D?" (id 0) (at 132.08 91.7574 90)
+    (property "Reference" "D3" (id 0) (at 132.08 91.7574 90)
       (effects (font (size 1.27 1.27)) (justify right))
     )
@@
   (symbol (lib_id "Device:LED") (at 171.45 91.44 90) (unit 1)
     (in_bom yes) (on_board yes) (fields_autoplaced)
-    (property "Reference" "D?" (id 0) (at 175.26 91.7574 90)
+    (property "Reference" "D4" (id 0) (at 175.26 91.7574 90)
       (effects (font (size 1.27 1.27)) (justify right))
     )
@@
   (symbol (lib_id "Device:R") (at 204.47 110.49 0) (unit 1)
     (in_bom yes) (on_board yes) (fields_autoplaced)
-    (property "Reference" "R?" (id 0) (at 207.01 109.2199 0)
+    (property "Reference" "R21" (id 0) (at 207.01 109.2199 0)
       (effects (font (size 1.27 1.27)) (justify left))
     )
@@
   (symbol (lib_id "power:+5V") (at 128.27 74.93 0) (unit 1)
     (in_bom yes) (on_board yes) (fields_autoplaced)
-    (property "Reference" "#PWR?" (id 0) (at 128.27 78.74 0)
+    (property "Reference" "#PWR029" (id 0) (at 128.27 78.74 0)
       (effects (font (size 1.27 1.27)) hide)
     )
@@
   (symbol (lib_id "Transistor_FET:AO3400A") (at 125.73 102.87 0) (unit 1)
     (in_bom yes) (on_board yes) (fields_autoplaced)
-    (property "Reference" "Q?" (id 0) (at 132.08 101.5999 0)
+    (property "Reference" "Q3" (id 0) (at 132.08 101.5999 0)
       (effects (font (size 1.27 1.27)) (justify left))
     )
@@
   (symbol (lib_id "Device:LED") (at 214.63 91.44 90) (unit 1)
     (in_bom yes) (on_board yes) (fields_autoplaced)
-    (property "Reference" "D?" (id 0) (at 218.44 91.7574 90)
+    (property "Reference" "D5" (id 0) (at 218.44 91.7574 90)
       (effects (font (size 1.27 1.27)) (justify right))
     )
@@
   (symbol (lib_id "Device:R") (at 128.27 81.28 0) (unit 1)
     (in_bom yes) (on_board yes) (fields_autoplaced)
-    (property "Reference" "R?" (id 0) (at 130.81 80.0099 0)
+    (property "Reference" "R18" (id 0) (at 130.81 80.0099 0)
       (effects (font (size 1.27 1.27)) (justify left))
     )
@@
   (symbol (lib_id "power:+5V") (at 171.45 74.93 0) (unit 1)
     (in_bom yes) (on_board yes) (fields_autoplaced)
-    (property "Reference" "#PWR?" (id 0) (at 171.45 78.74 0)
-      (effects (font (size 1.27 1.27)) hide)
-    )
+    (property "Reference" "#PWR031" (id 0) (at 171.45 78.74 0)
+      (effects (font (size 1.27 1.27)) hide)
+    )

Commit message: WIP
Parts:
- Q2, Q3, Q4, Q5: manf# (none) -> AO3400A
- R13: renamed from R15; footprint (none) -> Resistor_SMD:R_0603_1608Metric
- R14: renamed from R16; footprint (none) -> Resistor_SMD:R_0603_1608Metric
- R15: renamed from R17; footprint (none) -> Resistor_SMD:R_0603_1608Metric
- R16: renamed from R18; footprint (none) -> Resistor_SMD:R_0603_1608Metric
- R17: renamed from R19; footprint (none) -> Resistor_SMD:R_0603_1608Metric
- R18: renamed from R20; footprint (none) -> Resistor_SMD:R_0603_1608Metric
- R19: renamed from R21; footprint (none) -> Resistor_SMD:R_0603_1608Metric
- R20: renamed from R22; footprint (none) -> Resistor_SMD:R_0603_1608Metric
Other:
- title: Chrysler Scanner -> TJ Diag
Changed lines of the file:
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@@
   (paper "A4")
   (title_block
-    (title "Chrysler Scanner")
-    (date "2023-06-25")
-    (rev "V2.11")
+    (title "TJ Diag")
+    (date "2023-07-01")
+    (rev "V1.00")
     (company "andy@britishideas.com")
     (comment 1 "V210/ChryslerScanner_V210/schematic/ChryslerScanner_V210_schematic.pdf")
@@
   (symbol (lib_id "power:GND") (at 214.63 119.38 0) (unit 1)
     (in_bom yes) (on_board yes) (fields_autoplaced)
-    (property "Reference" "#PWR034" (id 0) (at 214.63 125.73 0)
+    (property "Reference" "#PWR030" (id 0) (at 214.63 125.73 0)
       (effects (font (size 1.27 1.27)) hide)
     )
@@
   (symbol (lib_id "power:GND") (at 171.45 119.38 0) (unit 1)
     (in_bom yes) (on_board yes) (fields_autoplaced)
-    (property "Reference" "#PWR032" (id 0) (at 171.45 125.73 0)
+    (property "Reference" "#PWR028" (id 0) (at 171.45 125.73 0)
       (effects (font (size 1.27 1.27)) hide)
     )
@@
   (symbol (lib_id "Device:R") (at 74.93 110.49 0) (unit 1)
     (in_bom yes) (on_board yes) (fields_autoplaced)
-    (property "Reference" "R15" (id 0) (at 77.47 109.2199 0)
+    (property "Reference" "R13" (id 0) (at 77.47 109.2199 0)
       (effects (font (size 1.27 1.27)) (justify left))
     )
@@
       (effects (font (size 1.27 1.27)) (justify left))
     )
-    (property "Footprint" "" (id 2) (at 73.152 110.49 90)
+    (property "Footprint" "Resistor_SMD:R_0603_1608Metric" (id 2) (at 73.152 110.49 90)
       (effects (font (size 1.27 1.27)) hide)
     )
@@
   (symbol (lib_id "Device:R") (at 161.29 110.49 0) (unit 1)
     (in_bom yes) (on_board yes) (fields_autoplaced)
-    (property "Reference" "R19" (id 0) (at 163.83 109.2199 0)
+    (property "Reference" "R17" (id 0) (at 163.83 109.2199 0)
       (effects (font (size 1.27 1.27)) (justify left))
     )
@@
       (effects (font (size 1.27 1.27)) (justify left))
     )
-    (property "Footprint" "" (id 2) (at 159.512 110.49 90)
+    (property "Footprint" "Resistor_SMD:R_0603_1608Metric" (id 2) (at 159.512 110.49 90)
       (effects (font (size 1.27 1.27)) hide)
     )
@@
   (symbol (lib_id "power:+5V") (at 214.63 74.93 0) (unit 1)
     (in_bom yes) (on_board yes) (fields_autoplaced)
-    (property "Reference" "#PWR033" (id 0) (at 214.63 78.74 0)
+    (property "Reference" "#PWR029" (id 0) (at 214.63 78.74 0)
       (effects (font (size 1.27 1.27)) hide)
     )
@@
       (effects (font (size 1.27 1.27)) (justify left) hide)
     )
+    (property "manf#" "AO3400A" (id 4) (at 82.55 102.87 0)
+      (effects (font (size 1.27 1.27)) hide)
+    )
     (pin "1")
     (pin "2")
@@
   (symbol (lib_id "power:GND") (at 128.27 119.38 0) (unit 1)
     (in_bom yes) (on_board yes) (fields_autoplaced)
-    (property "Reference" "#PWR030" (id 0) (at 128.27 125.73 0)
+    (property "Reference" "#PWR026" (id 0) (at 128.27 125.73 0)
       (effects (font (size 1.27 1.27)) hide)
     )
@@
   (symbol (lib_id "Device:R") (at 85.09 81.28 0) (unit 1)
     (in_bom yes) (on_board yes) (fields_autoplaced)
-    (property "Reference" "R16" (id 0) (at 87.63 80.0099 0)
+    (property "Reference" "R14" (id 0) (at 87.63 80.0099 0)
       (effects (font (size 1.27 1.27)) (justify left))
     )
@@
       (effects (font (size 1.27 1.27)) (justify left))
     )
-    (property "Footprint" "" (id 2) (at 83.312 81.28 90)
+    (property "Footprint" "Resistor_SMD:R_0603_1608Metric" (id 2) (at 83.312 81.28 90)
       (effects (font (size 1.27 1.27)) hide)
     )
@@
       (effects (font (size 1.27 1.27)) (justify left) hide)
     )
+    (property "manf#" "AO3400A" (id 4) (at 168.91 102.87 0)
+      (effects (font (size 1.27 1.27)) hide)
+    )
     (pin "1")
     (pin "2")
@@
       (effects (font (size 1.27 1.27)) (justify left) hide)
     )
+    (property "manf#" "AO3400A" (id 4) (at 212.09 102.87 0)
+      (effects (font (size 1.27 1.27)) hide)
+    )
     (pin "1")
     (pin "2")
@@
   (symbol (lib_id "power:+5V") (at 85.09 74.93 0) (unit 1)
     (in_bom yes) (on_board yes) (fields_autoplaced)
-    (property "Reference" "#PWR027" (id 0) (at 85.09 78.74 0)
+    (property "Reference" "#PWR023" (id 0) (at 85.09 78.74 0)
       (effects (font (size 1.27 1.27)) hide)
     )
@@
   (symbol (lib_id "power:GND") (at 85.09 119.38 0) (unit 1)
     (in_bom yes) (on_board yes) (fields_autoplaced)
-    (property "Reference" "#PWR028" (id 0) (at 85.09 125.73 0)
+    (property "Reference" "#PWR024" (id 0) (at 85.09 125.73 0)
       (effects (font (size 1.27 1.27)) hide)
     )
@@
   (symbol (lib_id "Device:R") (at 214.63 81.28 0) (unit 1)
     (in_bom yes) (on_board yes) (fields_autoplaced)
-    (property "Reference" "R22" (id 0) (at 217.17 80.0099 0)
+    (property "Reference" "R20" (id 0) (at 217.17 80.0099 0)
       (effects (font (size 1.27 1.27)) (justify left))
     )
@@
       (effects (font (size 1.27 1.27)) (justify left))
     )
-    (property "Footprint" "" (id 2) (at 212.852 81.28 90)
+    (property "Footprint" "Resistor_SMD:R_0603_1608Metric" (id 2) (at 212.852 81.28 90)
       (effects (font (size 1.27 1.27)) hide)
     )
@@
   (symbol (lib_id "Device:R") (at 171.45 81.28 0) (unit 1)
     (in_bom yes) (on_board yes) (fields_autoplaced)
-    (property "Reference" "R20" (id 0) (at 173.99 80.0099 0)
+    (property "Reference" "R18" (id 0) (at 173.99 80.0099 0)
       (effects (font (size 1.27 1.27)) (justify left))
     )
@@
       (effects (font (size 1.27 1.27)) (justify left))
     )
-    (property "Footprint" "" (id 2) (at 169.672 81.28 90)
+    (property "Footprint" "Resistor_SMD:R_0603_1608Metric" (id 2) (at 169.672 81.28 90)
       (effects (font (size 1.27 1.27)) hide)
     )
@@
   (symbol (lib_id "Device:R") (at 118.11 110.49 0) (unit 1)
     (in_bom yes) (on_board yes) (fields_autoplaced)
-    (property "Reference" "R17" (id 0) (at 120.65 109.2199 0)
+    (property "Reference" "R15" (id 0) (at 120.65 109.2199 0)
       (effects (font (size 1.27 1.27)) (justify left))
     )
@@
       (effects (font (size 1.27 1.27)) (justify left))
     )
-    (property "Footprint" "" (id 2) (at 116.332 110.49 90)
+    (property "Footprint" "Resistor_SMD:R_0603_1608Metric" (id 2) (at 116.332 110.49 90)
       (effects (font (size 1.27 1.27)) hide)
     )
@@
   (symbol (lib_id "Device:R") (at 204.47 110.49 0) (unit 1)
     (in_bom yes) (on_board yes) (fields_autoplaced)
-    (property "Reference" "R21" (id 0) (at 207.01 109.2199 0)
+    (property "Reference" "R19" (id 0) (at 207.01 109.2199 0)
       (effects (font (size 1.27 1.27)) (justify left))
     )
@@
       (effects (font (size 1.27 1.27)) (justify left))
     )
-    (property "Footprint" "" (id 2) (at 202.692 110.49 90)
+    (property "Footprint" "Resistor_SMD:R_0603_1608Metric" (id 2) (at 202.692 110.49 90)
       (effects (font (size 1.27 1.27)) hide)
     )
@@
   (symbol (lib_id "power:+5V") (at 128.27 74.93 0) (unit 1)
     (in_bom yes) (on_board yes) (fields_autoplaced)
-    (property "Reference" "#PWR029" (id 0) (at 128.27 78.74 0)
+    (property "Reference" "#PWR025" (id 0) (at 128.27 78.74 0)
       (effects (font (size 1.27 1.27)) hide)
     )
@@
       (effects (font (size 1.27 1.27)) (justify left) hide)
     )
+    (property "manf#" "AO3400A" (id 4) (at 125.73 102.87 0)
+      (effects (font (size 1.27 1.27)) hide)
+    )
     (pin "1")
     (pin "2")
@@
   (symbol (lib_id "Device:R") (at 128.27 81.28 0) (unit 1)
     (in_bom yes) (on_board yes) (fields_autoplaced)
-    (property "Reference" "R18" (id 0) (at 130.81 80.0099 0)
+    (property "Reference" "R16" (id 0) (at 130.81 80.0099 0)
       (effects (font (size 1.27 1.27)) (justify left))
     )
@@
       (effects (font (size 1.27 1.27)) (justify left))
     )
-    (property "Footprint" "" (id 2) (at 126.492 81.28 90)
+    (property "Footprint" "Resistor_SMD:R_0603_1608Metric" (id 2) (at 126.492 81.28 90)
       (effects (font (size 1.27 1.27)) hide)
     )
@@
   (symbol (lib_id "power:+5V") (at 171.45 74.93 0) (unit 1)
     (in_bom yes) (on_board yes) (fields_autoplaced)
-    (property "Reference" "#PWR031" (id 0) (at 171.45 78.74 0)
-      (effects (font (size 1.27 1.27)) hide)
-    )
+    (property "Reference" "#PWR027" (id 0) (at 171.45 78.74 0)
+      (effects (font (size 1.27 1.27)) hide)
+    )
