File: PCB/V210/ChryslerScanner_V210/OBDII.kicad_sch (KiCad schematic)
At the start: 5 parts, among them J2 SCI, J3 C-OBD-II-16M, J4 CCD, J5 PCI

Commit message: WIP
Parts:
- J2: footprint Connector_JST:JST_PH_B6B-PH-K_1x06_P2.00mm_Vertical -> Connector_PinHeader_2.54mm:PinHeader_1x06_P2.54mm_Vertical
- J4: footprint Connector_JST:JST_PH_B2B-PH-K_1x02_P2.00mm_Vertical -> Connector_PinHeader_2.54mm:PinHeader_1x02_P2.54mm_Vertical
- J5: footprint Connector_JST:JST_PH_B3B-PH-K_1x03_P2.00mm_Vertical -> Connector_PinHeader_2.54mm:PinHeader_1x03_P2.54mm_Vertical; manf# B3B-PH-KL -> (none)
Changed lines of the file:
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@@
     (property "Reference" "J4" (id 0) (at 158.75 48.26 0))
     (property "Value" "CCD" (id 1) (at 158.75 50.8 0))
-    (property "Footprint" "Connector_JST:JST_PH_B2B-PH-K_1x02_P2.00mm_Vertical" (id 2) (at 158.75 54.61 0)
+    (property "Footprint" "Connector_PinHeader_2.54mm:PinHeader_1x02_P2.54mm_Vertical" (id 2) (at 158.75 54.61 0)
       (effects (font (size 1.27 1.27)) hide)
     )
@@
     (property "Reference" "J2" (id 0) (at 104.14 43.18 0))
     (property "Value" "SCI" (id 1) (at 104.14 45.72 0))
-    (property "Footprint" "Connector_JST:JST_PH_B6B-PH-K_1x06_P2.00mm_Vertical" (id 2) (at 104.14 54.61 0)
+    (property "Footprint" "Connector_PinHeader_2.54mm:PinHeader_1x06_P2.54mm_Vertical" (id 2) (at 104.14 54.61 0)
       (effects (font (size 1.27 1.27)) hide)
     )
@@
     (property "Reference" "J5" (id 0) (at 198.12 46.99 0))
     (property "Value" "PCI" (id 1) (at 198.12 49.53 0))
-    (property "Footprint" "Connector_JST:JST_PH_B3B-PH-K_1x03_P2.00mm_Vertical" (id 2) (at 198.12 55.88 0)
+    (property "Footprint" "Connector_PinHeader_2.54mm:PinHeader_1x03_P2.54mm_Vertical" (id 2) (at 198.12 55.88 0)
       (effects (font (size 1.27 1.27)) hide)
     )
@@
       (effects (font (size 1.27 1.27)) hide)
     )
-    (property "manf#" "B3B-PH-KL" (id 4) (at 198.12 55.88 0)
+    (property "manf#" "" (id 4) (at 198.12 55.88 0)
       (effects (font (size 1.27 1.27)) hide)
     )
