File: PCB/V210/ChryslerScanner_V210/SCI.kicad_sch (KiCad schematic)
At the start: 30 parts, among them Q15 2N7002DW, Q16 2N7002DW, Q17 2N7002DW, U11 74LVC2G66, U12 74LVC2G66, U13 74LVC2G66

Commit message: WIP
Parts:
- C31, C32, C33, C34, C35, C36: footprint (none) -> Capacitor_SMD:C_0603_1608Metric
- Q7: renamed from Q15; footprint (none) -> Package_TO_SOT_SMD:SOT-363_SC-70-6; manf# (none) -> 2N7002DW
- Q8: renamed from Q16; footprint (none) -> Package_TO_SOT_SMD:SOT-363_SC-70-6; manf# (none) -> 2N7002DW
- Q9: renamed from Q17; footprint (none) -> Package_TO_SOT_SMD:SOT-363_SC-70-6; manf# (none) -> 2N7002DW
- R44: renamed from R66; footprint (none) -> Resistor_SMD:R_0603_1608Metric
- R45: renamed from R67; footprint (none) -> Resistor_SMD:R_0603_1608Metric
- R46: renamed from R68; footprint (none) -> Resistor_SMD:R_0603_1608Metric
- R47: renamed from R69; footprint (none) -> Resistor_SMD:R_0603_1608Metric
- R48: renamed from R70; footprint (none) -> Resistor_SMD:R_0603_1608Metric
- R49: renamed from R71; footprint (none) -> Resistor_SMD:R_0603_1608Metric
- R50: renamed from R72; footprint (none) -> Resistor_SMD:R_0603_1608Metric
- R51: renamed from R73; footprint (none) -> Resistor_SMD:R_0603_1608Metric
- R52: renamed from R74; footprint (none) -> Resistor_SMD:R_0603_1608Metric
- R53: renamed from R75; footprint (none) -> Resistor_SMD:R_0603_1608Metric
- R54: renamed from R76; footprint (none) -> Resistor_SMD:R_0603_1608Metric
- R55: renamed from R77; footprint (none) -> Resistor_SMD:R_0603_1608Metric
- R56: renamed from R78; footprint (none) -> Resistor_SMD:R_0603_1608Metric
- R57: renamed from R79; footprint (none) -> Resistor_SMD:R_0603_1608Metric
- R58: renamed from R80; footprint (none) -> Resistor_SMD:R_0603_1608Metric
- R59: renamed from R81; footprint (none) -> Resistor_SMD:R_0603_1608Metric
- R60: renamed from R82; footprint (none) -> Resistor_SMD:R_0603_1608Metric
- R61: renamed from R83; footprint (none) -> Resistor_SMD:R_0603_1608Metric
- U11, U12, U13: footprint (none) -> Package_SO:TSSOP-8_3x3mm_P0.65mm; manf# (none) -> 74LVC2G66DP,125
Other:
- title: Chrysler Scanner -> TJ Diag

Commit message: Added OBD-II connector.
Parts:
- renumbered C31 to C27, C32 to C28, C33 to C29, C34 to C30, C35 to C31, C36 to C32, R44 to R35, R45 to R36, R46 to R37, R47 to R38, R48 to R39, R49 to R40, R50 to R41, R51 to R42, R52 to R43, R53 to R44, R54 to R45, R55 to R46, R56 to R47, R57 to R48, R58 to R49, R59 to R50, R60 to R51, R61 to R52, U12 to U10, U13 to U11, U11 to U9

Commit message: Added CCD back in - needed for early TJs.
Parts:
- renumbered C27 to C30, C28 to C31, C29 to C32, C30 to C33, C31 to C34, C32 to C35, Q8 to Q10, Q9 to Q11, Q7 to Q9, R35 to R47, R36 to R48, R37 to R49, R38 to R50, R39 to R51, R40 to R52, R41 to R53, R42 to R54, R43 to R55, R44 to R56, R45 to R57, R46 to R58, R47 to R59, R48 to R60, R49 to R61, R50 to R62, R51 to R63, R52 to R64, U9 to U12, U10 to U13, U11 to U14
