File: PCB/V210/ChryslerScanner_V210/ChryslerScanner_V210.kicad_pcb (KiCad board)
At the start: 2 copper layers, 42 x 88.5 mm, 148 parts, among them J1 USB_B_Micro, J2 SCI, J3 C-OBD-II-16M, J4 CCD, J5 PCI, Q1 UMH3N, Q10 2N7002DW, Q11 2N7002DW, Q2 AO3400A, Q3 AO3400A, Q4 AO3400A, Q5 AO3400A, Q6 BSD235CH6327XTSA1, Q7 BSD235CH6327XTSA1, Q8 IRF7324, Q9 2N7002DW, SW1 RESET, SW2 BOOT, U1 ESP32-PICO-D4, U10 SN74LVC1G14DBV, U11 TS391RILT, U12 74LVC2G66, U13 74LVC2G66, U14 74LVC2G66, U2 PI4IOE5V6416ZDEX, U3 USBLC6-2SC6, U4 CP2102N-Axx-xQFN28, U5 NCV7808BDTRKG, U6 TLV76150DCYR, U7 TLV76133DCYR, U8 TS391RILT, U9 SN74LVC1G14DBV

Commit message: Working on PCB layout. Deleted old versions.
Parts:
- moved FID3 276.0 mm to (106.5, 57.1)
- moved FID1 274.7 mm to (106.5, 140.3)
- moved R35 241.0 mm to (134.7, 102.7), turned to 180 degrees
- moved R41 239.5 mm to (137.4, 117.3)
- moved D9 237.9 mm to (129.0, 114.6), turned to 90 degrees
- moved D11 234.8 mm to (134.2, 114.5), turned to 90 degrees
- moved R45 234.6 mm to (137.3, 114.4), turned to -90 degrees
- moved FID2 232.9 mm to (143.5, 140.3)
- moved R43 232.7 mm to (130.6, 114.8), turned to 90 degrees
- moved R36 230.3 mm to (136.5, 105.3), turned to 90 degrees
- moved R33 229.4 mm to (141.8, 96.2), turned to 180 degrees
- moved R46 228.3 mm to (143.9, 111.7), turned to 90 degrees
- moved R39 228.0 mm to (136.7, 121.3), turned to 90 degrees
- moved U10 227.7 mm to (134.9, 99.5), turned to -90 degrees
- moved C29 227.1 mm to (141.4, 114.1), turned to 180 degrees
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Other:
- board text added: "(C) andy@britishideas.com 2023 GPL V3"
- board text added: "BOOT"
- board text added: "RST"
- board text added: "TJ DIAG V1.0"

Commit message: Working on PCB layout.
Parts:
- moved FID3 27.3 mm to (128.0, 74.0)
- moved FID1 22.4 mm to (108.0, 118.0)
- moved FID2 7.72 mm to (141.0, 133.0)
- moved R8 3.20 mm to (130.5, 102.8)
- moved C11 1.60 mm to (127.3, 102.8)
- moved C12 1.60 mm to (128.9, 102.8)
- moved R64 0.14 mm to (143.5, 87.1), turned to 0 degrees
Routing:
- net +3V3: track 0.00 -> 277.2 mm, vias 0 -> 23
- net +5V: track 0.00 -> 223.2 mm, vias 0 -> 18
- net /OBDII/CCD+: track 0.00 -> 101.9 mm, vias 0 -> 5
- net /OBDII/CCD-: track 0.00 -> 93.9 mm, vias 0 -> 5
- net /MCU/RX0: track 0.00 -> 76.3 mm, vias 0 -> 4
- net /MCU/PCI_RX: track 0.00 -> 75.9 mm, vias 0 -> 6
- net /MCU/TX0: track 0.00 -> 73.2 mm, vias 0 -> 4
- net +12V: track 0.00 -> 71.2 mm, vias 0 -> 4
- net /OBDII/SCI_PCM_RX_A-6: track 0.00 -> 71.1 mm, vias 0 -> 5
- net /MCU/PCI_TX: track 0.00 -> 70.6 mm, vias 0 -> 8
- net /OBDII/SCI_TCM_TX_B-15: track 0.00 -> 63.4 mm, vias 0 -> 3
- net /OBDII/SCI_PCM_TX_AB_TCM_TX_A-7: track 0.00 -> 61.2 mm, vias 0 -> 2
- net /OBDII/SCI_PCM_RX_B-12: track 0.00 -> 61.1 mm, vias 0 -> 6
- net /OBDII/SCI_TCM_RX_A-14: track 0.00 -> 60.6 mm, vias 0 -> 3
- net /MCU/V_BA: track 0.00 -> 56.1 mm, vias 0 -> 6
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- added copper zone on B.Cu, net GND
- added copper zone on F.Cu, net GND
Other:
- outline, holes or cut-outs redrawn
- board text added: "Based on ChryslerScanner by László Dániel"
- board text added: "andy@britishideas.com GPL V3"
- board text removed: "(C) andy@britishideas.com 2023 GPL V3"

Commit message: Working on PCB layout.
Routing:
- net GND: vias 12 -> 55

Commit message: Working on PCB layout.
Connections:
- U1 pad 4: (no net) -> +3V3
- U1 pad 43: (no net) -> +3V3
- U1 pad 44: (no net) -> unconnected-(U1-Pad44)
- U1 pad 45: (no net) -> unconnected-(U1-Pad45)
- U1 pad 46: (no net) -> +3V3
- U1 pad 47: (no net) -> unconnected-(U1-Pad47)
- U1 pad 48: (no net) -> unconnected-(U1-Pad48)
Routing:
- net +3V3: track 277.2 -> 287.4 mm
- net /CCD/TBEN: track 31.5 -> 32.1 mm
- net GND: vias 55 -> 172

Commit message: Added Jeep TJ silhouette to bottom of board.
Parts:
- added G***: LOGO, ChryslerScanner:JeepSilhouette_40mm, B.Cu at (124.9, 97.9)
